Commit message: JointTrajectory seems to work

File: src/phantomx_description/urdf/phantomx.urdf (robot description, URDF)
Before this commit: robot PhantomX, 26 links, 25 joints
Joints:
- joint j_tibia_rr: limit lower=-2.6179939 upper=2.6179939 effort=2.8 velocity=2.6548668 -> lower=-2.6179939 upper=2.6179939 effort=0.9 velocity=2.6548668

Commit message: Changed urdf at xacro level

File: src/phantomx_description/urdf/phantomx.urdf (robot description, URDF)
Before this commit: robot PhantomX, 26 links, 25 joints
Joints:
- joint j_tibia_rr: limit lower=-2.6179939 upper=2.6179939 effort=0.9 velocity=2.6548668 -> lower=-2.6179939 upper=2.6179939 effort=2.8 velocity=2.6548668

File: src/phantomx_description/urdf/phantomx_urdf.xacro (robot description, xacro)
@@ -8,5 +8,5 @@
         <parent link="${parent}"/>
         <child link="MP_BODY"/>
-        <insert_block name="origin" />
+        <xacro:insert_block name="origin" />
       </joint>
       <link name="MP_BODY">
@@ -166,8 +166,7 @@
     <type>transmission_interface/SimpleTransmission</type>
     <joint name="j_c1_${suffix}">
-      <hardwareInterface>EffortJointInterface</hardwareInterface>
+      <hardwareInterface>hardware_interface/PositionJointInterface</hardwareInterface>
     </joint>
     <actuator name="m_c1_${suffix}">
-      <hardwareInterface>EffortJointInterface</hardwareInterface>
       <mechanicalReduction>1</mechanicalReduction>
     </actuator>
@@ -176,8 +175,7 @@
     <type>transmission_interface/SimpleTransmission</type>
     <joint name="j_thigh_${suffix}">
-      <hardwareInterface>EffortJointInterface</hardwareInterface>
+      <hardwareInterface>hardware_interface/PositionJointInterface</hardwareInterface>
     </joint>
     <actuator name="m_thigh_${suffix}">
-      <hardwareInterface>EffortJointInterface</hardwareInterface>
       <mechanicalReduction>1</mechanicalReduction>
     </actuator>
@@ -186,8 +184,7 @@
     <type>transmission_interface/SimpleTransmission</type>
     <joint name="j_tibia_${suffix}">
-      <hardwareInterface>EffortJointInterface</hardwareInterface>
+      <hardwareInterface>hardware_interface/PositionJointInterface</hardwareInterface>
     </joint>
     <actuator name="m_tibia_${suffix}">
-      <hardwareInterface>EffortJointInterface</hardwareInterface>
       <mechanicalReduction>1</mechanicalReduction>
     </actuator>

Commit message: Managed to remove robot sliding and jittering

File: src/phantomx_description/urdf/phantomx.urdf (robot description, URDF)
Before this commit: robot PhantomX, 26 links, 25 joints
Links:
- link c1_lf: mass 0.024357719 -> 0.012
- link c1_lm: mass 0.024357719 -> 0.012
- link c1_lr: mass 0.024357719 -> 0.012
- link c1_rf: mass 0.024357719 -> 0.012
- link c1_rm: mass 0.024357719 -> 0.012
- link c1_rr: mass 0.024357719 -> 0.012
- link c2_lf: mass 0.024357719 -> 0.012
- link c2_lm: mass 0.024357719 -> 0.012
- link c2_lr: mass 0.024357719 -> 0.012
- link c2_rf: mass 0.024357719 -> 0.012
- link c2_rm: mass 0.024357719 -> 0.012
- link c2_rr: mass 0.024357719 -> 0.012
- link thigh_lf: mass 0.024357719 -> 0.070
- link thigh_lm: mass 0.024357719 -> 0.070
- link thigh_lr: mass 0.024357719 -> 0.070
- link thigh_rf: mass 0.024357719 -> 0.070
- link thigh_rm: mass 0.024357719 -> 0.070
- link thigh_rr: mass 0.024357719 -> 0.070
- link tibia_lf: mass 0.024357719 -> 0.080
- link tibia_lm: mass 0.024357719 -> 0.080
- link tibia_lr: mass 0.024357719 -> 0.080
- link tibia_rf: mass 0.024357719 -> 0.080
- link tibia_rm: mass 0.024357719 -> 0.080
- link tibia_rr: mass 0.024357719 -> 0.080

File: src/phantomx_description/urdf/phantomx_urdf.xacro (robot description, xacro)
@@ -14,5 +14,5 @@
           <origin xyz="0 0 0" />
           <mass value="0.97559947"/>
-          <inertia ixx="3.1081800"  ixy="-0.25460189"  ixz="2.0318174" iyy="6.3787776" iyz="0.16417863" izz="5.3316425" />
+          <inertia ixx="0.004"  ixy="0"  ixz="0" iyy="0.004" iyz="0" izz="0.004" />
         </inertial>
         <visual>
@@ -48,6 +48,6 @@
     <inertial>
       <origin xyz="0 -${connect_offset} 0" rpy="0 0 0"  />
-      <mass value="0.024357719"/>
-     <inertia ixx="0.0051411124"  ixy="-0.00057530255"  ixz="-0.000024729049" iyy="0.0081915737" iyz="-0.000019223094" izz="0.0011379812" />
+      <mass value="0.012"/>
+      <inertia ixx="0.0005"  ixy="0"  ixz="0" iyy="0.0005" iyz="0" izz="0.0005" />
     </inertial>
     <visual>
@@ -71,6 +71,6 @@
     <inertial>
       <origin xyz="0 -${connect_offset} 0" rpy="0 0 0"  />
-      <mass value="0.024357719"/>
-     <inertia ixx="0.0051411124"  ixy="-0.00057530255"  ixz="-0.000024729049" iyy="0.0081915737" iyz="-0.000019223094" izz="0.0011379812" />
+      <mass value="0.012"/>
+      <inertia ixx="0.0005"  ixy="0"  ixz="0" iyy="0.0005" iyz="0" izz="0.0005" />
     </inertial>
     <visual>
@@ -94,6 +94,6 @@
     <inertial>
       <origin xyz="0 0 0" rpy="0 0 0"  />
-      <mass value="0.024357719"/>
-     <inertia ixx="0.0051411124"  ixy="-0.00057530255"  ixz="-0.000024729049" iyy="0.0081915737" iyz="-0.000019223094" izz="0.0011379812" />
+      <mass value="0.070"/>
+      <inertia ixx="0.0005"  ixy="0"  ixz="0" iyy="0.0005" iyz="0" izz="0.0005" />
     </inertial>
     <visual>
@@ -117,6 +117,6 @@
     <inertial>
       <origin xyz="0 0 0" rpy="0 0 0"  />
-      <mass value="0.024357719"/>
-     <inertia ixx="0.0051411124"  ixy="-0.00057530255"  ixz="-0.000024729049" iyy="0.0081915737" iyz="-0.000019223094" izz="0.0011379812" />
+      <mass value="0.080"/>
+      <inertia ixx="0.0005"  ixy="0"  ixz="0" iyy="0.0005" iyz="0" izz="0.0005" />
     </inertial>
     <visual>
@@ -201,4 +201,6 @@
   <gazebo reference="tibia_${suffix}">
     <material>Gazebo/Grey</material>
+    <mu1 value="12000.0"/>
+    <mu2 value="12000.0"/>
   </gazebo>
 </xacro:macro>

Commit message: Testing with tibia_rm's mass = 5kg

File: src/phantomx_description/urdf/phantomx.urdf (robot description, URDF)
Before this commit: robot PhantomX, 26 links, 25 joints
Links:
- link tibia_rm: mass 0.080 -> 5.080

Commit message: Using walker code to generate gait trajectories

File: src/phantomx_description/urdf/phantomx.urdf (robot description, URDF)
Before this commit: robot PhantomX, 26 links, 25 joints
Links:
- link tibia_rm: mass 5.080 -> 0.080
